File: alpacESP-PCB/alpacESP-PCB.kicad_sch (KiCad schematic)
At the start: 35 parts, among them U0 ESP32-S3-WROOM-1U

Commit message: added more components
Parts:
- added C? (x3): 1uF, symbol Device:C
- added D?: B340, Diode_SMD:D_SMC, symbol Diode:B340
- added J? (x5): A2501WV-3P, kicad-parts:A2501WV-3P, symbol keyboard_parts:A2501WV-3P
- added J? (x6): A2501WV-2P, kicad-parts:A2501WV-2P, symbol keyboard_parts:A2501WV-2P
- added J?: EXP1, symbol Connector_Generic:Conn_02x05_Odd_Even
- added J? (x4): Conn_01x03_Male, symbol Connector:Conn_01x03_Male
- added J?: EXP2, symbol Connector_Generic:Conn_02x05_Odd_Even
- added Q? (x3): 2N7002, Package_TO_SOT_SMD:SOT-23, symbol Transistor_FET:2N7002
- added R? (x6): 4.7K, symbol Device:R
- added R? (x3): 10K, symbol Device:R
- added R? (x3): 100K, symbol Device:R
- added R?: 3K, symbol Device:R
- added U?: EL817, Package_DIP:DIP-4_W7.62mm, symbol Isolator:EL817
Connections:
- net 3V3: now also R?.1, R?.2, R?.2, R?.2
- net 5V: now also D?.2 (A), J?.1, J?.1 (Pin_1), J?.1 (Pin_1), J?.1 (Pin_1), J?.1 (Pin_1), J?.2 (Pin_2), J?.3, R?.2
- net GND: now also C?.1, C?.1, C?.1, J?.1, J?.1, J?.1, J?.1, J?.1 (Pin_1), J?.2, J?.2, J?.2, J?.2, J?.2 (Pin_2), Q?.2 (S), Q?.2 (S), Q?.2 (S), R?.1, R?.1, R?.1, U?.3
- new net: J?.1, J?.2 (Pin_2) (x3)
- new net: J?.2, Q?.3 (D) (x3)
- new net: Q?.1 (G), R?.1, R?.2 (x3)
- new net: R?.1, U?.1
- new net 4V7: D?.1 (K), J?.3, J?.3, J?.3, R?.2, R?.2
- new net BLTOUCH: J?.3 (Pin_3)
- new net EN_RESET: J?.3 (Pin_3)
- new net FAN0: R?.2
- new net FAN1: R?.2
- new net FAN2: R?.2
- new net FAN_IN: J?.3 (Pin_3), J?.3 (Pin_3), J?.3 (Pin_3)
- new net LCD_BTN: J?.9 (Pin_9)
- new net LCD_BTN1: J?.8 (Pin_8)
- new net LCD_BTN2: J?.6 (Pin_6)
- new net LCD_D4: J?.6 (Pin_6)
- new net LCD_EN: J?.8 (Pin_8)
- new net LCD_RS: J?.7 (Pin_7)
- new net RGB: J?.2
- new net RUNOUT: J?.3
- new net TEMP0: C?.2, J?.1, R?.1
- new net TEMP1: C?.2, J?.1, R?.1
- new net TEMP_BED: C?.2, J?.1, R?.1
- new net X_MIN: J?.2, R?.1
- new net Y_MIN: J?.2, R?.1
- new net Z_MIN: J?.2, U?.2
- new net Z_MIN_L: R?.2, U?.4
Other:
- moved on the sheet: C?, Q?, R?, SW?, U0, U?

Commit message: Dead
Parts:
- added C?: 100uF, symbol Device:C
- added D? (x3): LED, symbol Device:LED
- added J? (x3): KF129-5.08-2P, kicad-parts:KF129-5.08-2P, symbol keyboard_parts:KF129-5.08-2P
- added J? (x2): Conn_01x08_Female, symbol Connector:Conn_01x08_Female
- added J? (x3): A2501WV-2P, kicad-parts:A2501WV-2P, symbol keyboard_parts:A2501WV-2P
- added J? (x3): Conn_01x03_Male, symbol Connector:Conn_01x03_Male
- added J?: HX25003-4A, kicad-parts:A2501WV-4P, symbol keyboard_parts:HX25003-4A
- added Q? (x3): 2N7002, Package_TO_SOT_SMD:SOT-23, symbol Transistor_FET:2N7002
- added R? (x3): 1K, symbol Device:R
- added R? (x3): 20K, symbol Device:R
- added R? (x3): 100K, symbol Device:R
Connections:
- net 4V7: now also J?.2 (Pin_2)
- net 5V: now also J?.1 (Pin_1), J?.1 (Pin_1), J?.1 (Pin_1)
- net FAN_IN: now also J?.3 (Pin_3), J?.3 (Pin_3), J?.3 (Pin_3)
- net GND: now also C?.2, J?.1 (Pin_1), J?.2, J?.2, J?.2, J?.7 (Pin_7), Q?.2 (S), Q?.2 (S), Q?.2 (S), R?.2, R?.2, R?.2
- new net: D?.1 (K), J?.2, Q?.3 (D) (x3)
- new net: D?.2 (A), R?.2 (x3)
- new net: Q?.1 (G), R?.1, R?.2 (x3)
- new net: J?.3 (Pin_3), J?.4
- new net: J?.3, J?.4 (Pin_4)
- new net: J?.2, J?.5 (Pin_5)
- new net: J?.1, J?.6 (Pin_6)
- new net: J?.1, J?.2 (Pin_2) (x3)
- new net HEAT0: R?.1
- new net HEAT1: R?.1
- new net HEATBED_IN: J?.1, R?.1
- new net HEAT_BED: R?.1
- new net HOT_IN: J?.1, J?.1, R?.1, R?.1
- new net MOTOR_IN: C?.1, J?.8 (Pin_8)
